File: 3bitflashadc.kicad_sch (KiCad schematic)
At the start: 0 parts

Commit message: added major components, wirings to be fixed
Parts:
- added AFF1: LTS-6960HR, Display_7Segment:7SegmentLED_LTS6760_LTS6780, symbol Display_Character:LTS-6960HR
- added C2, C4: 100nf, symbol Device:C
- added R1, R2, R3, R4, R5, R6, R7, R8: R, symbol Device:R
- added R10, R11, R12, R13, R14, R15, R9: 10k, Display_7Segment:7SegmentLED_LTS6760_LTS6780, symbol Device:R
- added RV1: R_Potentiometer, Package_SO:TSSOP-20_4.4x6.5mm_P0.65mm, symbol Device:R_Potentiometer
- added Ra, Rb, Rc, Rd, Re, Rf, Rg: (no value), Display_7Segment:7SegmentLED_LTS6760_LTS6780, symbol Device:R
- added U1, U1E, U2, U2E: LM339, Package_TO_SOT_SMD:SOT-23-5, symbol Comparator:LM339
- added U3: 74148, Package_DIP:DIP-20_W7.62mm, symbol 74xx_IEEE:74148
- added U4: 74LS04, Package_SO:SOIC-20W_7.5x12.8mm_P1.27mm, symbol 74xx:74LS04
- added U5: 7447, Package_CSP:Xilinx_CSG48_7.0x7.0mm_Layout7x7_P0.8mm, symbol 74xx_IEEE:7447
Connections:
- new net: RV1.2, U1.10 (-), U1.4 (-), U1.6 (-), U1.8 (-), U2.10 (-), U2.4 (-), U2.6 (-)
- new net: R4.1, R5.2, U1.9 (+)
- new net: R6.1, R7.2, U2.7 (+)
- new net: R3.1, R4.2, U1.11 (+)
- new net: R7.1, R8.1, U2.11 (+)
- new net: AFF1.4 (c), Rc.2
- new net: AFF1.1 (e), Re.2
- new net: AFF1.10 (g), Rg.2
- new net: AFF1.2 (d), Rd.2
- new net: AFF1.6 (b), Rb.2
- new net: AFF1.7 (a), Ra.2
- new net: AFF1.9 (f), Rf.2
- new net: R2.1, R3.2, U1.7 (+)
- new net: R1.1, R2.2, U1.5 (+)
- new net: R5.1, R6.2, U2.5 (+)
- new net 5V: C2.2, C4.2, R1.2, R10.2, R11.2, R12.2, R13.2, R14.2, R15.2, R9.2, RV1.1, U1E.5 (+), U2E.7 (+), U3.16 (VCC), U5.16 (VCC), U5.3 (~{LT}), U5.4 (~{BI}), U5.5 (~{RBI})
- new net GND: C2.1, C4.1, R8.2, RV1.3, U1E.4 (-), U2E.6 (-), U3.10 (~{IO}), U3.5 (~{EI}), U5.6 (D)
- new net U1A: R9.1, U1.2, U3.4 (~{I7})
- new net U1B: R10.1, U1.1, U3.3 (~{I6})
- new net U1C: R11.1, U1.13, U3.2 (~{I5})
- new net U1D: R12.1, U1.14, U3.1 (~{I4})
- new net U2A: R13.1, U2.2, U3.13 (~{I3})
- new net U2B: R14.1, U2.1, U3.12 (~{I2})
- new net U2C: R15.1, U2.13, U3.11 (~{I1})

Commit message: Global label issue needs to be fixed, but the footprints are all assigned
Parts:
- removed U1E, U2E: LM339, Package_TO_SOT_SMD:SOT-23-5, symbol Comparator:LM339
- added unit 5 of U1
- added unit 5 of U2
- added unit 7 of U4
- C2, C4: footprint (none) -> Capacitor_THT:C_Disc_D3.4mm_W2.1mm_P2.50mm
- R1, R2, R3, R4, R5, R6, R7, R8: value R -> 1k; footprint (none) -> Resistor_THT:R_Axial_DIN0207_L6.3mm_D2.5mm_P7.62mm_Horizontal
- R10, R11, R12, R13, R14, R15, R9: footprint Display_7Segment:7SegmentLED_LTS6760_LTS6780 -> Resistor_THT:R_Axial_DIN0207_L6.3mm_D2.5mm_P7.62mm_Horizontal
- RV1: value R_Potentiometer -> 10k; footprint Package_SO:TSSOP-20_4.4x6.5mm_P0.65mm -> Potentiometer_THT:Potentiometer_Alpha_RD901F-40-00D_Single_Vertical
- Ra1: renamed from Ra; value (none) -> 220; footprint Display_7Segment:7SegmentLED_LTS6760_LTS6780 -> Resistor_THT:R_Axial_DIN0207_L6.3mm_D2.5mm_P7.62mm_Horizontal
- Rb1: renamed from Rb; value (none) -> 220; footprint Display_7Segment:7SegmentLED_LTS6760_LTS6780 -> Resistor_THT:R_Axial_DIN0207_L6.3mm_D2.5mm_P7.62mm_Horizontal
- Rc1: renamed from Rc; value (none) -> 220; footprint Display_7Segment:7SegmentLED_LTS6760_LTS6780 -> Resistor_THT:R_Axial_DIN0207_L6.3mm_D2.5mm_P7.62mm_Horizontal
- Rd1: renamed from Rd; value (none) -> 220; footprint Display_7Segment:7SegmentLED_LTS6760_LTS6780 -> Resistor_THT:R_Axial_DIN0207_L6.3mm_D2.5mm_P7.62mm_Horizontal
- Re1: renamed from Re; value (none) -> 220; footprint Display_7Segment:7SegmentLED_LTS6760_LTS6780 -> Resistor_THT:R_Axial_DIN0207_L6.3mm_D2.5mm_P7.62mm_Horizontal
- Rf1: renamed from Rf; value (none) -> 220; footprint Display_7Segment:7SegmentLED_LTS6760_LTS6780 -> Resistor_THT:R_Axial_DIN0207_L6.3mm_D2.5mm_P7.62mm_Horizontal
- Rg1: renamed from Rg; value (none) -> 220; footprint Display_7Segment:7SegmentLED_LTS6760_LTS6780 -> Resistor_THT:R_Axial_DIN0207_L6.3mm_D2.5mm_P7.62mm_Horizontal
- U1, U2: footprint Package_TO_SOT_SMD:SOT-23-5 -> Package_DIP:CERDIP-14_W7.62mm_SideBrazed_LongPads
- U3: footprint Package_DIP:DIP-20_W7.62mm -> Package_DIP:CERDIP-14_W7.62mm_SideBrazed_LongPads
- U4: footprint Package_SO:SOIC-20W_7.5x12.8mm_P1.27mm -> Package_DIP:CERDIP-14_W7.62mm_SideBrazed_LongPads
- U5: footprint Package_CSP:Xilinx_CSG48_7.0x7.0mm_Layout7x7_P0.8mm -> Package_DIP:CERDIP-16_W7.62mm_SideBrazed_Socket
Connections:
- net 5V: now also AFF1.3 (C.A.), AFF1.8 (C.A.), U1.3 (V+), U2.3 (V+), U4.14 (VCC)
- net GND: now also U3.8 (GND), U5.8 (GND), U1.12 (V-), U2.12 (V-), U4.7 (GND)
- net at U4.3: now also U3.7 (~{S1})
- net at U4.4: now also U5.1 (B)
- net at Rc1.1: now also U5.11 (~{c})
- net at U4.1: now also U3.9 (~{S0})
- net at U4.2: now also U5.7 (A)
- net at Rg1.1: now also U5.14 (~{g})
- net at Rb1.1: now also U5.12 (~{b})
- net at Re1.1: now also U5.9 (~{e})
- net at Rf1.1: now also U5.15 (~{f})
- net at U5.10 (~{d}): now also Rd1.1
- net at U5.13 (~{a}): now also Ra1.1
- net at U5.2 (C): now also U4.6
- net at U3.6 (~{S2}): now also U4.5
- net U1A renamed UA1
- net U1B renamed UB1
- net U1C renamed UC1
- net U1D renamed UD1
- net U2A renamed UA2
- net U2B renamed UB2
- net U2C renamed UC2
- no-connect marks 0 -> 3
Other:
- moved on the sheet: AFF1, U4A, U4B, U4C

Commit message: Completed schematic, still need to be inspected
Parts:
- added C3: 100nf, Capacitor_THT:C_Disc_D3.4mm_W2.1mm_P2.50mm, symbol Device:C
- added J1: ExternalPower, TerminalBlock:TerminalBlock_MaiXu_MX126-5.0-02P_1x02_P5.00mm, symbol Connector:Screw_Terminal_01x02
- added unit 4 of U2
- added unit 4 of U4
- added unit 6 of U4
- added unit 5 of U4
- U3: footprint Package_DIP:CERDIP-14_W7.62mm_SideBrazed_LongPads -> Package_DIP:CERDIP-16_W7.62mm_SideBrazed_LongPads
Connections:
- net 5V: now also C3.2, J1.2 (Pin_2)
- net GND: now also C3.1, J1.1 (Pin_1), U2.8 (-), U2.9 (+), U4.11, U4.13, U4.9
- net UA1: no longer names the net of R9.1, U1.2, U3.4 (~{I7})
- net UA2: no longer names the net of R13.1, U2.2, U3.13 (~{I3})
- net UB1: no longer names the net of R10.1, U1.1, U3.3 (~{I6})
- net UB2: no longer names the net of R14.1, U2.1, U3.12 (~{I2})
- net UC1: no longer names the net of R11.1, U1.13, U3.2 (~{I5})
- net UC2: no longer names the net of R15.1, U2.13, U3.11 (~{I1})
- net UD1: no longer names the net of R12.1, U1.14, U3.1 (~{I4})
- no-connect marks 3 -> 7
Other:
- note added: "Board Power"
- note added: "ICs Power"
- note added: "Unused IC pins (connected to GND to avoid oscillation)"
- moved on the sheet: R1, R10, R11, R12, R13, R14, R15, R2, R3, R4, R5, R6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

Commit message: Done with the schematic and working with the PCB routing
Parts:
- removed C2: 100nf, Capacitor_THT:C_Disc_D3.4mm_W2.1mm_P2.50mm, symbol Device:C
- removed U3: 74148, Package_DIP:CERDIP-16_W7.62mm_SideBrazed_LongPads, symbol 74xx_IEEE:74148
- added C5, C6, C7, C8, C9: 100nf, Capacitor_THT:C_Disc_D3.4mm_W2.1mm_P2.50mm, symbol Device:C
- added R16, R17: 1k, Resistor_THT:R_Axial_DIN0207_L6.3mm_D2.5mm_P7.62mm_Horizontal, symbol Device:R
- added R18, R19: 10k, Resistor_THT:R_Axial_DIN0207_L6.3mm_D2.5mm_P7.62mm_Horizontal, symbol Device:R
- added U3: LM339, Package_DIP:CERDIP-14_W7.62mm_SideBrazed_LongPads_Socket, symbol Comparator:LM339
- added U6: 74147, Package_DIP:CERDIP-16_W7.62mm_SideBrazed_Socket, symbol 74xx_IEEE:74147
- U1, U2, U4: footprint Package_DIP:CERDIP-14_W7.62mm_SideBrazed_LongPads -> Package_DIP:CERDIP-14_W7.62mm_SideBrazed_LongPads_Socket
Connections:
- net 5V: now also C5.2, C6.2, C7.2, C8.2, C9.2, R18.2, R19.2, U3.3 (V+), U6.16 (VCC)
- net GND: now also C5.1, C6.1, C7.1, C8.1, C9.1, R17.2, U3.10 (-), U3.11 (+), U3.12 (V-), U3.6 (-), U3.7 (+), U3.8 (-), U3.9 (+), U6.8 (GND); no longer R8.2, U2.8 (-), U2.9 (+), U4.9, U5.6 (D)
- net 1D: now reaches R12.1, U1.14
- net 1D: now also U6.3 (~{E6})
- net at RV1.2, U1.10 (-), U1.4 (-)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: now also U2.8 (-), U3.4 (-)
- net 2B: now reaches R14.1, U2.1
- net 2B: now also U6.1 (~{E4})
- net at U4.3: now also U6.7 (~{S1})
- net B: now reaches U4.4, U5.1 (B)
- net 1C: now reaches R11.1, U1.13
- net 1C: now also U6.4 (~{E7})
- net 2C: now reaches R15.1, U2.13
- net 2C: now also U6.13 (~{E3})
- net at U4.1: now also U6.9 (~{S0})
- net A: now reaches U4.2, U5.7 (A)
- net 2D: now reaches U2.14
- net 2D: now also R18.1, U6.12 (~{E2})
- net D: now reaches U4.8
- net D: now also U5.6 (D)
- net 2A: now reaches R13.1, U2.2
- net 2A: now also U6.2 (~{E5})
- net 1B: now reaches R10.1, U1.1
- net 1B: now also U6.5 (~{E8})
- net C: now reaches U4.6, U5.2 (C)
- net 1A: now reaches R9.1, U1.2
- net 1A: now also U6.10 (~{E9})
- net at U4.5: now also U6.6 (~{S2})
- new net: R16.1, R8.2, U2.9 (+)
- new net: U4.9, U6.14 (~{S3})
- new net: R16.2, R17.1, U3.5 (+)
- new net 3A: R19.1, U3.2, U6.11 (~{E1})
- no-connect marks 7 -> 6
Other:
- moved on the sheet: AFF1, C3, C4, J1, R1, R10, R11, R12, R13, R14, R15, R2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
